Commit message: Cambio descripcion URDF

File: examen_description/urdf/scara_urdf.xacro (robot description, xacro)
@@ -92,5 +92,5 @@
         <limit lower="-3.14159" upper="3.14159" velocity="50.0"
                effort="1000.0"/>
-        <origin xyz="0.075 0 0.1" rpy="0 0 0"/>
+        <origin xyz="0 0 0.1" rpy="0 0 0"/>
     </joint>
     <link name="link_3">
@@ -123,5 +123,5 @@
         <limit lower="-3.14159" upper="3.14159" velocity="50.0"
                effort="1000.0"/>
-        <origin xyz="0.05 0.0 0.5" rpy="0 0 0"/>
+        <origin xyz="0.0 0.0 0.5" rpy="0 0 0"/>
     </joint>
     <link name="link_4">
@@ -154,5 +154,5 @@
         <limit lower="-3.14159" upper="3.14159" velocity="50.0"
                effort="1000.0"/>
-        <origin xyz="0.05 0.0 0.5" rpy="0 0 0"/>
+        <origin xyz="0 0.0 0.5" rpy="0 0 0"/>
     </joint>
 </robot>

Commit message: Correccion ejes de rotacion

File: examen_description/urdf/scara_urdf.xacro (robot description, xacro)
@@ -89,5 +89,5 @@
         <parent link="link_1"/>
         <child link="link_2"/>
-        <axis xyz="1 0 0"/>
+        <axis xyz="0 1 0"/>
         <limit lower="-3.14159" upper="3.14159" velocity="50.0"
                effort="1000.0"/>
@@ -120,5 +120,5 @@
         <parent link="link_2"/>
         <child link="link_3"/>
-        <axis xyz="1 0 0"/>
+        <axis xyz="0 1 0"/>
         <limit lower="-3.14159" upper="3.14159" velocity="50.0"
                effort="1000.0"/>
@@ -151,5 +151,5 @@
         <parent link="link_3"/>
         <child link="link_4"/>
-        <axis xyz="1 0 0"/>
+        <axis xyz="0 1 0"/>
         <limit lower="-3.14159" upper="3.14159" velocity="50.0"
                effort="1000.0"/>

Commit message: Correcciones URDF para movilidad real

File: examen_description/urdf/scara_urdf.xacro (robot description, xacro)
@@ -1,5 +1,5 @@
 <?xml version="1.0" encoding="utf-8"?>
-<!--Aqui comienza el robot-->
-<robot name="robot_scara" xmlns:xacro="http://ros.org/wiki/xacro" >
+<!-- Aquí comienza el robot -->
+<robot name="robot_scara" xmlns:xacro="http://ros.org/wiki/xacro">
     <link name="world">
     </link>
@@ -13,5 +13,5 @@
             <origin xyz="0.0 0.0 0.025" rpy="0 0 0" />
             <geometry>
-                <box size="0.3 0.3 0.05" />
+                <box size="0.4 0.4 0.05" />
             </geometry>
             <material name="grey">
@@ -22,5 +22,5 @@
             <origin xyz="0.0 0.0 0.025" rpy="0 0 0" />
             <geometry>
-                <box size="0.3 0.3 0.05" />
+                <box size="0.4 0.4 0.05" />
             </geometry>
         </collision>
@@ -36,5 +36,5 @@
             <origin xyz="0.0 0.0 0.05" rpy="0 0 0" />
             <geometry>
-                <box size="0.1 0.1 0.1" />
+                <box size="0.15 0.15 0.1" />
             </geometry>
             <material name="red">
@@ -45,5 +45,5 @@
             <origin xyz="0.0 0.0 0.05" rpy="0 0 0" />
             <geometry>
-                <box size="0.05 0.05 0.1" />
+                <box size="0.15 0.15 0.1" />
             </geometry>
         </collision>
@@ -65,5 +65,5 @@
     <link name="link_2">
         <visual>
-            <origin xyz="0.0 0.0 0.25" rpy="0 0 0" />
+            <origin xyz="0.0 0.025 0.25" rpy="0 0 0" />
             <geometry>
                 <box size="0.05 0.05 0.5" />
@@ -74,5 +74,5 @@
         </visual>
         <collision>
-            <origin xyz="0.0 0.0 0.25" rpy="0 0 0" />
+            <origin xyz="0.0 0.025 0.25" rpy="0 0 0" />
             <geometry>
                 <box size="0.05 0.05 0.5" />
@@ -92,9 +92,9 @@
         <limit lower="-3.14159" upper="3.14159" velocity="50.0"
                effort="1000.0"/>
-        <origin xyz="0 0 0.1" rpy="0 0 0"/>
+        <origin xyz="0 0.075 0.1" rpy="0 0 0"/>
     </joint>
     <link name="link_3">
         <visual>
-            <origin xyz="0.0 0.0 0.25" rpy="0 0 0" />
+            <origin xyz="0.0 -0.025 0.25" rpy="0 0 0" />
             <geometry>
                 <box size="0.05 0.05 0.5" />
@@ -105,5 +105,5 @@
         </visual>
         <collision>
-            <origin xyz="0.0 0.0 0.25" rpy="0 0 0" />
+            <origin xyz="0.0 -0.025 0.25" rpy="0 0 0" />
             <geometry>
                 <box size="0.05 0.05 0.5" />
@@ -154,5 +154,22 @@
         <limit lower="-3.14159" upper="3.14159" velocity="50.0"
                effort="1000.0"/>
-        <origin xyz="0 0.0 0.5" rpy="0 0 0"/>
+        <origin xyz="0 -0.075 0.5" rpy="0 0 0"/>
+    </joint>
+    <!-- Sistema de referencia en la punta de link_4 -->
+    <link name="link_4_tip">
+        <visual>
+            <origin xyz="0 0 0.15" rpy="0 0 0"/>
+            <geometry>
+                <sphere radius="0.01"/>
+            </geometry>
+            <material name="yellow">
+                <color rgba="1.0 1.0 0.0 1.0"/>
+            </material>
+        </visual>
+    </link>
+    <joint name="link_4_tip_joint" type="fixed">
+        <parent link="link_4"/>
+        <child link="link_4_tip"/>
+        <origin xyz="0 0 0.3" rpy="0 0 0"/>
     </joint>
 </robot>
